Commit message: 更新URDF，删除mujoco中的contact_callback函数

File: robot_description/galileo_mini15_description/urdf/robot.urdf (robot description, URDF)
Before this commit: robot JLL_ROBOT, 17 links, 16 joints
Links:
- link FL_abd_link: geometry collision mesh filename=package://galileo_mini15_description/meshes/FL_abd_link.STL scale=1 1 1; visual mesh filename=package://galileo_mini15_description/meshes/FL_abd_link.STL scale=1 1 1
- link FL_hip_link: geometry collision mesh filename=package://galileo_mini15_description/meshes/FL_hip_link.STL scale=1 1 1; visual mesh filename=package://galileo_mini15_description/meshes/FL_hip_link.STL scale=1 1 1
- link FL_knee_link: geometry collision mesh filename=package://galileo_mini15_description/meshes/FL_knee_link.STL scale=1 1 1; visual mesh filename=package://galileo_mini15_description/meshes/FL_knee_link.STL scale=1 1 1
- link FR_abd_link: geometry collision mesh filename=package://galileo_mini15_description/meshes/FL_abd_link.STL scale=1.0 -1.0 1.0; visual mesh filename=package://galileo_mini15_description/meshes/FL_abd_link.STL scale=1.0 -1.0 1.0
- link FR_hip_link: geometry collision mesh filename=package://galileo_mini15_description/meshes/FL_hip_link.STL scale=1.0 -1.0 1.0; visual mesh filename=package://galileo_mini15_description/meshes/FL_hip_link.STL scale=1.0 -1.0 1.0
- link FR_knee_link: geometry collision mesh filename=package://galileo_mini15_description/meshes/FL_knee_link.STL scale=1.0 -1.0 1.0; visual mesh filename=package://galileo_mini15_description/meshes/FL_knee_link.STL scale=1.0 -1.0 1.0
- link HL_abd_link: geometry collision mesh filename=package://galileo_mini15_description/meshes/RL_abd_link.STL scale=1 1 1; visual mesh filename=package://galileo_mini15_description/meshes/RL_abd_link.STL scale=1 1 1
- link HL_hip_link: geometry collision mesh filename=package://galileo_mini15_description/meshes/RL_hip_link.STL scale=1 1 1; visual mesh filename=package://galileo_mini15_description/meshes/RL_hip_link.STL scale=1 1 1
- link HL_knee_link: geometry collision mesh filename=package://galileo_mini15_description/meshes/RL_knee_link.STL scale=1 1 1; visual mesh filename=package://galileo_mini15_description/meshes/RL_knee_link.STL scale=1 1 1
- link HR_abd_link: geometry collision mesh filename=package://galileo_mini15_description/meshes/RL_abd_link.STL scale=1.0 -1.0 1.0; visual mesh filename=package://galileo_mini15_description/meshes/RL_abd_link.STL scale=1.0 -1.0 1.0
- link HR_hip_link: geometry collision mesh filename=package://galileo_mini15_description/meshes/RL_hip_link.STL scale=1.0 -1.0 1.0; visual mesh filename=package://galileo_mini15_description/meshes/RL_hip_link.STL scale=1.0 -1.0 1.0
- link HR_knee_link: geometry collision mesh filename=package://galileo_mini15_description/meshes/RL_knee_link.STL scale=1.0 -1.0 1.0; visual mesh filename=package://galileo_mini15_description/meshes/RL_knee_link.STL scale=1.0 -1.0 1.0
- link base_link: mass 9.2006 -> 16.057; geometry collision mesh filename=package://galileo_mini15_description/meshes/trunk.STL scale=1 1 1; visual mesh filename=package://galileo_mini15_description/meshes/trunk.STL scale=1 1 1

Commit message: 更新galileo_mini15的xml

File: robot_description/galileo_mini15_description/urdf/robot.urdf (robot description, URDF)
Before this commit: robot galileo_mini15, 17 links, 16 joints
Links:
- added link world
Joints:
- added joint floating_base_joint: type floating, parent world, child base_link, origin xyz=0 0 0 rpy=0 0 0
- joint FL_hip_joint: limit lower=-1.0472 upper=4.1888 effort=100 velocity=21 -> lower=-4.1888 upper=1.0472 effort=100 velocity=21
- joint FR_hip_joint: limit lower=-1.0472 upper=4.1888 effort=100 velocity=21 -> lower=-4.1888 upper=1.0472 effort=100 velocity=21
- joint HL_hip_joint: limit lower=-1.0472 upper=4.1888 effort=100 velocity=21 -> lower=-4.1888 upper=1.0472 effort=100 velocity=21
- joint HR_hip_joint: limit lower=-1.0472 upper=4.1888 effort=100 velocity=21 -> lower=-4.1888 upper=1.0472 effort=100 velocity=21
