Commit message: Change targetpose iteration from the current pose to the desired pose

File: robot_description/galileo_mini_description/urdf/robot.urdf (robot description, URDF)
Before this commit: robot galileo_mini_description, 18 links, 17 joints
Joints:
- joint FL_calf_joint: limit lower=-2.6965 upper=-0.9163 effort=150 velocity=21 -> lower=0.9163 upper=2.6965 effort=150 velocity=21
- joint FL_thigh_joint: limit lower=-4.1888 upper=1.0472 effort=100 velocity=21 -> lower=-1.0472 upper=4.1888 effort=100 velocity=21
- joint FR_calf_joint: limit lower=-2.6965 upper=-0.9163 effort=150 velocity=21 -> lower=0.9163 upper=2.6965 effort=150 velocity=21
- joint FR_thigh_joint: limit lower=-4.1888 upper=1.0472 effort=100 velocity=21 -> lower=-1.0472 upper=4.1888 effort=100 velocity=21
- joint RL_calf_joint: limit lower=-2.6965 upper=-0.9163 effort=150 velocity=21 -> lower=0.9163 upper=2.6965 effort=150 velocity=21
- joint RL_thigh_joint: limit lower=-4.1888 upper=1.0472 effort=100 velocity=21 -> lower=-1.0472 upper=4.1888 effort=100 velocity=21
- joint RR_calf_joint: limit lower=-2.6965 upper=-0.9163 effort=150 velocity=21 -> lower=0.9163 upper=2.6965 effort=150 velocity=21
- joint RR_thigh_joint: limit lower=-4.1888 upper=1.0472 effort=100 velocity=21 -> lower=-1.0472 upper=4.1888 effort=100 velocity=21

File: robot_description/simple_quadruped/urdf/simple_quadruped.urdf (robot description, URDF)
Before this commit: robot simple_quadruped, 17 links, 16 joints
Links:
- link FL_foot: geometry collision sphere radius=0.030; visual sphere radius=0.030
- link FR_foot: geometry collision sphere radius=0.030; visual sphere radius=0.030
- link RL_foot: geometry collision sphere radius=0.030; visual sphere radius=0.030
- link RR_foot: geometry collision sphere radius=0.030; visual sphere radius=0.030
Joints:
- joint FL_calf_joint: axis 0 -1 0 -> 0 1 0
- joint FL_thigh_joint: axis 0 -1 0 -> 0 1 0
- joint FR_calf_joint: axis 0 -1 0 -> 0 1 0
- joint FR_thigh_joint: axis 0 -1 0 -> 0 1 0
- joint RL_calf_joint: axis 0 -1 0 -> 0 1 0
- joint RL_thigh_joint: axis 0 -1 0 -> 0 1 0
- joint RR_calf_joint: axis 0 -1 0 -> 0 1 0
- joint RR_thigh_joint: axis 0 -1 0 -> 0 1 0

Commit message: 修改了urdf和xml文件格式

File: robot_description/galileo_mini_description/urdf/robot.urdf (robot description, URDF)
Before this commit: robot galileo_mini_description, 18 links, 17 joints
Links:
- removed link FL_calf
- removed link FL_foot
- removed link FL_hip
- removed link FL_thigh
- removed link FR_calf
- removed link FR_foot
- removed link FR_hip
- removed link FR_thigh
- removed link RL_calf
- removed link RL_foot
- removed link RL_hip
- removed link RL_thigh
- removed link RR_calf
- removed link RR_foot
- removed link RR_hip
- removed link RR_thigh
- removed link trunk
- removed link world
- added link FL_abd_link, mass 2.86; collision mesh filename=package://galileo_mini_description/meshes/FL_abd_link.STL; visual mesh filename=package://galileo_mini_description/meshes/FL_abd_link.STL
- added link FL_foot_link, mass 0.00020487; collision mesh filename=package://galileo_mini_description/meshes/FL_foot_link.STL; visual mesh filename=package://galileo_mini_description/meshes/FL_foot_link.STL
- added link FL_hip_link, mass 2.6; collision mesh filename=package://galileo_mini_description/meshes/FL_hip_link.STL; visual mesh filename=package://galileo_mini_description/meshes/FL_hip_link.STL
- added link FL_knee_link, mass 0.314; collision mesh filename=package://galileo_mini_description/meshes/FL_knee_link.STL; visual mesh filename=package://galileo_mini_description/meshes/FL_knee_link.STL
- added link FR_abd_link, mass 2.86; collision mesh filename=package://galileo_mini_description/meshes/FR_abd_link.STL; visual mesh filename=package://galileo_mini_description/meshes/FR_abd_link.STL
- added link FR_foot_link, mass 0.00020487; collision mesh filename=package://galileo_mini_description/meshes/FR_foot_link.STL; visual mesh filename=package://galileo_mini_description/meshes/FR_foot_link.STL
- added link FR_hip_link, mass 2.6; collision mesh filename=package://galileo_mini_description/meshes/FR_hip_link.STL; visual mesh filename=package://galileo_mini_description/meshes/FR_hip_link.STL
- added link FR_knee_link, mass 0.314; collision mesh filename=package://galileo_mini_description/meshes/FR_knee_link.STL; visual mesh filename=package://galileo_mini_description/meshes/FR_knee_link.STL
- added link HL_abd_link, mass 2.86; collision mesh filename=package://galileo_mini_description/meshes/HL_abd_link.STL; visual mesh filename=package://galileo_mini_description/meshes/HL_abd_link.STL
- added link HL_foot_link, mass 0.000204873572147578; collision mesh filename=package://galileo_mini_description/meshes/HL_foot_link.STL; visual mesh filename=package://galileo_mini_description/meshes/HL_foot_link.STL
- added link HL_hip_link, mass 2.6; collision mesh filename=package://galileo_mini_description/meshes/HL_hip_link.STL; visual mesh filename=package://galileo_mini_description/meshes/HL_hip_link.STL
- added link HL_knee_link, mass 0.314; collision mesh filename=package://galileo_mini_description/meshes/HL_knee_link.STL; visual mesh filename=package://galileo_mini_description/meshes/HL_knee_link.STL
- added link HR_abd_link, mass 2.86; collision mesh filename=package://galileo_mini_description/meshes/HR_abd_link.STL; visual mesh filename=package://galileo_mini_description/meshes/HR_abd_link.STL
- added link HR_foot_link, mass 0.000204873572147578; collision mesh filename=package://galileo_mini_description/meshes/HR_foot_link.STL; visual mesh filename=package://galileo_mini_description/meshes/HR_foot_link.STL
- added link HR_hip_link, mass 2.6; collision mesh filename=package://galileo_mini_description/meshes/HR_hip_link.STL; visual mesh filename=package://galileo_mini_description/meshes/HR_hip_link.STL
- added link HR_knee_link, mass 0.314; collision mesh filename=package://galileo_mini_description/meshes/HR_knee_link.STL; visual mesh filename=package://galileo_mini_description/meshes/HR_knee_link.STL
- added link base_link, mass 20.8; collision mesh filename=package://galileo_mini_description/meshes/base_link.STL; visual mesh filename=package://galileo_mini_description/meshes/base_link.STL
Joints:
- removed joint FL_calf_joint
- removed joint FL_thigh_joint
- removed joint FR_calf_joint
- removed joint FR_thigh_joint
- removed joint RL_calf_joint
- removed joint RL_foot_joint
- removed joint RL_hip_joint
- removed joint RL_thigh_joint
- removed joint RR_calf_joint
- removed joint RR_foot_joint
- removed joint RR_hip_joint
- removed joint RR_thigh_joint
- removed joint floating_base_joint
- added joint FL_abd_joint: type revolute, parent base_link, child FL_abd_link, origin xyz=0.2015 0.08 0 rpy=0 0 0, axis 1 0 0, limit lower=-0.80285 upper=0.80285 effort=100 velocity=21
- added joint FL_knee_joint: type revolute, parent FL_hip_link, child FL_knee_link, origin xyz=0 0 -0.26 rpy=0 0 0, axis 0 1 0, limit lower=-2.6965 upper=-0.9163 effort=150 velocity=21
- added joint FR_abd_joint: type revolute, parent base_link, child FR_abd_link, origin xyz=0.2015 -0.08 0 rpy=0 0 0, axis 1 0 0, limit lower=-0.80285 upper=0.80285 effort=100 velocity=21
- added joint FR_knee_joint: type revolute, parent FR_hip_link, child FR_knee_link, origin xyz=0 0 -0.26 rpy=0 0 0, axis 0 1 0, limit lower=-2.6965 upper=-0.9163 effort=150 velocity=21
- added joint HL_abd_joint: type revolute, parent base_link, child HL_abd_link, origin xyz=-0.2015 0.08 0 rpy=0 0 0, axis 1 0 0, limit lower=-0.80285 upper=0.80285 effort=100 velocity=21
- added joint HL_foot_joint: type fixed, parent HL_knee_link, child HL_foot_link, origin xyz=0.0329385085367515 0 -0.261492891464613 rpy=0 0 0, axis 0 0 0
- added joint HL_hip_joint: type revolute, parent HL_abd_link, child HL_hip_link, origin xyz=-0.1 0.1065 0 rpy=0 0 0, axis 0 1 0, limit lower=-1.0472 upper=4.1888 effort=100 velocity=21
- added joint HL_knee_joint: type revolute, parent HL_hip_link, child HL_knee_link, origin xyz=6.3209E-05 0 -0.26 rpy=0 0 0, axis 0 1 0, limit lower=-2.6965 upper=-0.9163 effort=150 velocity=21
- added joint HR_abd_joint: type revolute, parent base_link, child HR_abd_link, origin xyz=-0.2015 -0.08 0 rpy=0 0 0, axis 1 0 0, limit lower=-0.80285 upper=0.80285 effort=100 velocity=21
- added joint HR_foot_joint: type fixed, parent HR_knee_link, child HR_foot_link, origin xyz=0.032939 0 -0.26149 rpy=0 0 0, axis 0 0 0
- added joint HR_hip_joint: type revolute, parent HR_abd_link, child HR_hip_link, origin xyz=-0.1 -0.0934 0 rpy=0 0 0, axis 0 1 0, limit lower=-1.0472 upper=4.1888 effort=100 velocity=21
- added joint HR_knee_joint: type revolute, parent HR_hip_link, child HR_knee_link, origin xyz=0 0 -0.26 rpy=0 0 0, axis 0 1 0, limit lower=-2.6965 upper=-0.9163 effort=150 velocity=21
- joint FL_foot_joint: child FL_foot -> FL_foot_link; parent FL_calf -> FL_knee_link
- joint FL_hip_joint: axis 1 0 0 -> 0 1 0; child FL_hip -> FL_hip_link; limit lower=-0.80285 upper=0.80285 effort=100 velocity=21 -> lower=-1.0472 upper=4.1888 effort=100 velocity=21; origin xyz=0.2015 0.08 0 rpy=0 0 0 -> xyz=0.1 0.1065 0 rpy=0 0 0; parent trunk -> FL_abd_link
- joint FR_foot_joint: child FR_foot -> FR_foot_link; parent FR_calf -> FR_knee_link
- joint FR_hip_joint: axis 1 0 0 -> 0 1 0; child FR_hip -> FR_hip_link; limit lower=-0.80285 upper=0.80285 effort=100 velocity=21 -> lower=-1.0472 upper=4.1888 effort=100 velocity=21; origin xyz=0.2015 -0.08 0 rpy=0 0 0 -> xyz=0.1 -0.10685 0 rpy=0 0 0; parent trunk -> FR_abd_link

File: robot_description/galileo_mini_description/xacro/robot.xacro (robot description, xacro)
@@ -1,892 +1,491 @@
 <?xml version="1.0"?>
-<robot name="galileo_mini_description" xmlns:xacro="http://www.ros.org/wiki/xacro">
+<robot name="galileo_mini_description"
+  xmlns:xacro="http://www.ros.org/wiki/xacro">
   <xacro:include filename="$(find galileo_mini_description)/xacro/ros2_control.xacro" />
-  <!-- <xacro:include filename="$(find b2_description)/xacro/transmission.xacro" /> -->
-  <link name="base" />
-  <joint name="floating_base_joint" type="fixed">
-    <origin xyz="0 0 0" rpy="0 0 0" />
-    <parent link="base" />
-    <child link="trunk" />
-  </joint>
-  <link name="trunk">
-    <inertial>
-      <origin
-        xyz="0.03738 -0.0065903 0.0057934"
-        rpy="0 0 0" />
-      <mass
-        value="20.8" />
-      <inertia
-        ixx="0.131102"
-        ixy="0.001924"
-        ixz="0.001299"
-        iyy="0.407915"
-        iyz="0.002595"
-        izz="0.476755" />
-    </inertial>
-    <visual>
-      <origin
-        xyz="0 0 0"
-        rpy="0 0 0" />
-      <geometry>
-        <mesh
-          filename="package://galileo_mini_description/meshes/trunk.STL" />
-      </geometry>
-      <material
-        name="">
-        <color
-          rgba="0.75294 0.75294 0.75294 1" />
-      </material>
-    </visual>
-    <collision>
-      <origin
-        xyz="0 0 0" rpy="0 0 0" />
-      <geometry>
-        <box size="0.45 0.25 0.1" />
-      </geometry>
-    </collision>
-  </link>
-  <link name="FL_hip">
-    <inertial>
-      <origin
-        xyz="0.067568 0.0095934 1.3738E-05"
-        rpy="0 0 0" />
-      <mass
-        value="2.86" />
-      <inertia
-        ixx="0.004368"
-        ixy="0.000362"
-        ixz="0.000114"
-        iyy="0.007476"
-        iyz="0.000035"
-        izz="0.006777" />
-    </inertial>
-    <visual>
-      <origin
-        xyz="0 0 0"
-        rpy="0 0 0" />
-      <geometry>
-        <mesh
-          filename="package://galileo_mini_description/meshes/FL_hip.STL" />
-      </geometry>
-      <material
-        name="">
-        <color
-          rgba="0.75294 0.75294 0.75294 1" />
-      </material>
-    </visual>
-    <collision>
-      <origin
-        xyz="0.1 0.03325 0"
-        rpy="1.5707963 0 0" />
-      <geometry>
-        <cylinder radius="0.06" length="0.1065" />
+  <link name="base_link">
+    <inertial>
+      <origin xyz="0.03738 -0.0065903 0.0057934" rpy="0 0 0" />
+      <mass value="20.8" />
+      <inertia ixx="0.131102" ixy="0.001924" ixz="0.001299" iyy="0.407915" iyz="0.002595" izz="0.476755" />
+    </inertial>
+    <visual>
+      <origin xyz="0 0 0" rpy="0 0 0" />
+      <geometry>
+        <mesh filename="package://galileo_mini_description/meshes/base_link.STL" />
+      </geometry>
+      <material name="">
+        <color rgba="0.75294 0.75294 0.75294 1" />
+      </material>
+    </visual>
+    <collision>
+      <origin xyz="0 0 0" rpy="0 0 0" />
+      <geometry>
+        <mesh filename="package://galileo_mini_description/meshes/base_link.STL" />
+      </geometry>
+    </collision>
+  </link>
+  <!-- ****************************FR**************************** -->
+  <link name="FR_abd_link">
+    <inertial>
+      <origin xyz="0.067568 -0.0091759 -0.00023747" rpy="0 0 0" />
+      <mass value="2.86" />
+      <inertia ixx="0.004373" ixy="-0.000397" ixz="-0.000096" iyy="0.007483" iyz="0.000030" izz="0.006775" />
+    </inertial>
+    <visual>
+      <origin xyz="0 0 0" rpy="0 0 0" />
+      <geometry>
+        <mesh filename="package://galileo_mini_description/meshes/FR_abd_link.STL" />
+      </geometry>
+      <material name="">
+        <color rgba="0.75294 0.75294 0.75294 1" />
+      </material>
+    </visual>
+    <collision>
+      <origin xyz="0 0 0" rpy="0 0 0" />
+      <geometry>
+        <mesh filename="package://galileo_mini_description/meshes/FR_abd_link.STL" />
+      </geometry>
+    </collision>
+  </link>
+  <joint name="FR_abd_joint" type="revolute">
+    <origin xyz="0.2015 -0.08 0" rpy="0 0 0" />
+    <parent link="base_link" />
+    <child link="FR_abd_link" />
+    <axis xyz="1 0 0" />
+    <limit lower="-0.80285" upper="0.80285" effort="100" velocity="21" />
+  </joint>
+  <link name="FR_hip_link">
+    <inertial>
+      <origin xyz="-0.0095338 0.026092 -0.067392" rpy="0 0 0" />
+      <mass value="2.6" />
+      <inertia ixx="0.016261" ixy="0.000284" ixz="0.001143" iyy="0.016389" iyz="0.002508" izz="0.002194" />
+    </inertial>
+    <visual>
+      <origin xyz="0 0 0" rpy="0 0 0" />
+      <geometry>
+        <mesh filename="package://galileo_mini_description/meshes/FR_hip_link.STL" />
+      </geometry>
+      <material name="">
+        <color rgba="0.75294 0.75294 0.75294 1" />
+      </material>
+    </visual>
+    <collision>
+      <origin xyz="0 0 0" rpy="0 0 0" />
+      <geometry>
+        <mesh filename="package://galileo_mini_description/meshes/FR_hip_link.STL" />
+      </geometry>
+    </collision>
+  </link>
+  <joint name="FR_hip_joint" type="revolute">
+    <origin xyz="0.1 -0.10685 0" rpy="0 0 0" />
+    <parent link="FR_abd_link" />
+    <child link="FR_hip_link" />
+    <axis xyz="0 1 0" />
+    <limit upper="4.1888" lower="-1.0472" effort="100" velocity="21" />
+  </joint>
+  <link name="FR_knee_link">
+    <inertial>
+      <origin xyz="0.017829 -1.577E-05 -0.099213" rpy="0 0 0" />
+      <mass value="0.314" />
+      <inertia ixx="0.003733" ixy="-0.000000087" ixz="-0.0006" iyy="0.003882" iyz="0.000000838" izz="0.000177" />
+    </inertial>
+    <visual>
+      <origin xyz="0 0 0" rpy="0 0 0" />
+      <geometry>
+        <mesh filename="package://galileo_mini_description/meshes/FR_knee_link.STL" />
+      </geometry>
+      <material name="">
+        <color rgba="0.75294 0.75294 0.75294 1" />
+      </material>
+    </visual>
+    <collision>
+      <origin xyz="0 0 0" rpy="0 0 0" />
+      <geometry>
+        <mesh filename="package://galileo_mini_description/meshes/FR_knee_link.STL" />
+      </geometry>
+    </collision>
+  </link>
+  <joint name="FR_knee_joint" type="revolute">
+    <origin xyz="0 0 -0.26" rpy="0 0 0" />
+    <parent link="FR_hip_link" />
+    <child link="FR_knee_link" />
+    <axis xyz="0 1 0" />
+    <limit upper="-0.9163" lower="-2.6965" effort="150" velocity="21" />
+  </joint>
+  <link name="FR_foot_link">
+    <inertial>
+      <origin xyz="0 0 0" rpy="0 0 0" />
+      <mass value="0.00020487" />
+      <inertia ixx="1.096E-09" ixy="0" ixz="1.7152E-40" iyy="1.096E-09" iyz="0" izz="1.096E-09" />
+    </inertial>
+    <visual>
+      <origin xyz="0 0 0" rpy="0 0 0" />
+      <geometry>
+        <mesh filename="package://galileo_mini_description/meshes/FR_foot_link.STL" />
+      </geometry>
+      <material name="">
+        <color rgba="1 1 1 1" />
+      </material>
+    </visual>
+    <collision>
+      <origin xyz="0 0 0" rpy="0 0 0" />
+      <geometry>
+        <mesh filename="package://galileo_mini_description/meshes/FR_foot_link.STL" />
+      </geometry>
+    </collision>
+  </link>
+  <joint name="FR_foot_joint" type="fixed" dont_collapse="true">
+    <origin xyz="0.032939 0 -0.26149" rpy="0 0 0" />
+    <parent link="FR_knee_link" />
+    <child link="FR_foot_link" />
+    <axis xyz="0 0 0" />
+  </joint>
+  <!-- ****************************HR**************************** -->
+  <link name="HR_abd_link">
+    <inertial>
+      <origin xyz="-0.067556 -0.0095934 -1.7463E-05" rpy="0 0 0" />
+      <mass value="2.86" />
+      <inertia ixx="0.004372" ixy="0.000364" ixz="-0.000106" iyy="0.007471" iyz="-0.000038" izz="0.006768" />
+    </inertial>
+    <visual>
+      <origin xyz="0 0 0" rpy="0 0 0" />
+      <geometry>
+        <mesh filename="package://galileo_mini_description/meshes/HR_abd_link.STL" />
+      </geometry>
+      <material name="">
+        <color rgba="0.75294 0.75294 0.75294 1" />
+      </material>
+    </visual>
+    <collision>
+      <origin xyz="0 0 0" rpy="0 0 0" />
+      <geometry>
+        <mesh filename="package://galileo_mini_description/meshes/HR_abd_link.STL" />
+      </geometry>
+    </collision>
+  </link>
+  <joint name="HR_abd_joint" type="revolute">
+    <origin xyz="-0.2015 -0.08 0" rpy="0 0 0" />
+    <parent link="base_link" />
+    <child link="HR_abd_link" />
+    <axis xyz="1 0 0" />
+    <limit lower="-0.80285" upper="0.80285" effort="100" velocity="21" />
+  </joint>
+  <link name="HR_hip_link">
+    <inertial>
+      <origin xyz="-0.0098055 0.020667 -0.067167" rpy="0 0 0" />
+      <mass value="2.6" />
+      <inertia ixx="0.017144" ixy="0.000198" ixz="0.001067" iyy="0.016508" iyz="0.002833" izz="0.002907" />
+    </inertial>
+    <visual>
+      <origin xyz="0 0 0" rpy="0 0 0" />
+      <geometry>
+        <mesh filename="package://galileo_mini_description/meshes/HR_hip_link.STL" />
+      </geometry>
+      <material name="">
+        <color rgba="0.75294 0.75294 0.75294 1" />
+      </material>
+    </visual>
+    <collision>
+      <origin xyz="0 0 0" rpy="0 0 0" />
+      <geometry>
+        <mesh filename="package://galileo_mini_description/meshes/HR_hip_link.STL" />
+      </geometry>
+    </collision>
+  </link>
+  <joint name="HR_hip_joint" type="revolute">
+    <origin xyz="-0.1 -0.0934 0" rpy="0 0 0" />
+    <parent link="HR_abd_link" />
+    <child link="HR_hip_link" />
+    <axis xyz="0 1 0" />
+    <limit upper="4.1888" lower="-1.0472" effort="100" velocity="21" />
+  </joint>
+  <link name="HR_knee_link">
+    <inertial>
+      <origin xyz="0.017829 -1.577E-05 -0.099213" rpy="0 0 0" />
+      <mass value="0.314" />
+      <inertia ixx="0.003733" ixy="-0.000000087" ixz="-0.0006" iyy="0.003882" iyz="0.000000838" izz="0.000177" />
+    </inertial>
+    <visual>
+      <origin xyz="0 0 0" rpy="0 0 0" />
+      <geometry>
+        <mesh filename="package://galileo_mini_description/meshes/HR_knee_link.STL" />
+      </geometry>
+      <material name="">
+        <color rgba="0.75294 0.75294 0.75294 1" />
+      </material>
+    </visual>
+    <collision>
+      <origin xyz="0 0 0" rpy="0 0 0" />
+      <geometry>
+        <mesh filename="package://galileo_mini_description/meshes/HR_knee_link.STL" />
+      </geometry>
+    </collision>
+  </link>
+  <joint name="HR_knee_joint" type="revolute">
+    <origin xyz="0 0 -0.26" rpy="0 0 0" />
+    <parent link="HR_hip_link" />
+    <child link="HR_knee_link" />
+    <axis xyz="0 1 0" />
+    <limit upper="-0.9163" lower="-2.6965" effort="150" velocity="21" />
+  </joint>
+  <link name="HR_foot_link">
+    <inertial>
+      <origin xyz="0 0 0" rpy="0 0 0" />
+      <mass value="0.000204873572147578" />
+      <inertia ixx="1.09600066619755E-09" ixy="0" ixz="5.28443143791483E-42" iyy="1.09600066619755E-09" iyz="0" izz="1.09600066619755E-09" />
+    </inertial>
+    <visual>
+      <origin xyz="0 0 0" rpy="0 0 0" />
+      <geometry>
+        <mesh filename="package://galileo_mini_description/meshes/HR_foot_link.STL" />
+      </geometry>
+      <material name="">
+        <color rgba="1 1 1 1" />
+      </material>
+    </visual>
+    <collision>
+      <origin xyz="0 0 0" rpy="0 0 0" />
+      <geometry>
+        <mesh filename="package://galileo_mini_description/meshes/HR_foot_link.STL" />
+      </geometry>
+    </collision>
+  </link>
+  <joint name="HR_foot_joint" type="fixed" dont_collapse="true">
+    <origin xyz="0.032939 0 -0.26149" rpy="0 0 0" />
+    <parent link="HR_knee_link" />
+    <child link="HR_foot_link" />
+    <axis xyz="0 0 0" />
+  </joint>
+  <!-- ****************************FL**************************** -->
+  <link name="FL_abd_link">
+    <inertial>
+      <origin xyz="0.067568 0.0095934 1.3738E-05" rpy="0 0 0" />
+      <mass value="2.86" />
+      <inertia ixx="0.004368" ixy="0.000362" ixz="0.000114" iyy="0.007476" iyz="0.000035" izz="0.006777" />
+    </inertial>
+    <visual>
+      <origin xyz="0 0 0" rpy="0 0 0" />
+      <geometry>
+        <mesh filename="package://galileo_mini_description/meshes/FL_abd_link.STL" />
+      </geometry>
+      <material name="">
+        <color rgba="0.75294 0.75294 0.75294 1" />
+      </material>
+    </visual>
+    <collision>
+      <origin xyz="0 0 0" rpy="0 0 0" />
+      <geometry>
+        <mesh filename="package://galileo_mini_description/meshes/FL_abd_link.STL" />
+      </geometry>
+    </collision>
+  </link>
+  <joint name="FL_abd_joint" type="revolute">
+    <origin xyz="0.2015 0.08 0" rpy="0 0 0" />
+    <parent link="base_link" />
+    <child link="FL_abd_link" />
+    <axis xyz="1 0 0" />
+    <limit lower="-0.80285" upper="0.80285" effort="100" velocity="21" />
+  </joint>
+  <link name="FL_hip_link">
+    <inertial>
+      <origin xyz="-0.0090988 -0.0065295 -0.0688" rpy="0 0 0" />
+      <mass value="2.6" />
+      <inertia ixx="0.016848" ixy="-0.000310" ixz="0.001116" iyy="0.016749" iyz="-0.002270" izz="0.002088" />
+    </inertial>
+    <visual>
+      <origin xyz="0 0 0" rpy="0 0 0" />
+      <geometry>
+        <mesh filename="package://galileo_mini_description/meshes/FL_hip_link.STL" />
+      </geometry>
+      <material name="">
+        <color rgba="0.75294 0.75294 0.75294 1" />
+      </material>
+    </visual>
+    <collision>
+      <origin xyz="0 0 0" rpy="0 0 0" />
+      <geometry>
+        <mesh filename="package://galileo_mini_description/meshes/FL_hip_link.STL" />
       </geometry>
     </collision>
   </link>
   <joint name="FL_hip_joint" type="revolute">
-    <origin
-      xyz="0.2015 0.08 0"
-      rpy="0 0 0" />
-    <parent
-      link="trunk" />
-    <child
-      link="FL_hip" />
-    <axis
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