Commit message: 修改了urdf和xml文件格式

File: robot_description/galileo_mini_description/xacro/ros2_control.xacro (robot description, xacro)
@@ -5,4 +5,14 @@
             <plugin>hardware_mujoco/HardwareMujoco</plugin>
         </hardware>
+        <joint name="FR_abd_joint">
+            <command_interface name="position" />
+            <command_interface name="velocity" />
+            <command_interface name="effort" />
+            <command_interface name="kp" />
+            <command_interface name="kd" />
+            <state_interface name="position" />
+            <state_interface name="velocity" />
+            <state_interface name="effort" />
+        </joint>
         <joint name="FR_hip_joint">
             <command_interface name="position" />
@@ -15,5 +25,5 @@
             <state_interface name="effort" />
         </joint>
-        <joint name="FR_thigh_joint">
+        <joint name="FR_knee_joint">
             <command_interface name="position" />
             <command_interface name="velocity" />
@@ -25,5 +35,35 @@
             <state_interface name="effort" />
         </joint>
-        <joint name="FR_calf_joint">
+        <joint name="HR_abd_joint">
+            <command_interface name="position" />
+            <command_interface name="velocity" />
+            <command_interface name="effort" />
+            <command_interface name="kp" />
+            <command_interface name="kd" />
+            <state_interface name="position" />
+            <state_interface name="velocity" />
+            <state_interface name="effort" />
+        </joint>
+        <joint name="HR_hip_joint">
+            <command_interface name="position" />
+            <command_interface name="velocity" />
+            <command_interface name="effort" />
+            <command_interface name="kp" />
+            <command_interface name="kd" />
+            <state_interface name="position" />
+            <state_interface name="velocity" />
+            <state_interface name="effort" />
+        </joint>
+        <joint name="HR_knee_joint">
+            <command_interface name="position" />
+            <command_interface name="velocity" />
+            <command_interface name="effort" />
+            <command_interface name="kp" />
+            <command_interface name="kd" />
+            <state_interface name="position" />
+            <state_interface name="velocity" />
+            <state_interface name="effort" />
+        </joint>
+        <joint name="FL_abd_joint">
             <command_interface name="position" />
             <command_interface name="velocity" />
@@ -45,5 +85,5 @@
             <state_interface name="effort" />
         </joint>
-        <joint name="FL_thigh_joint">
+        <joint name="FL_knee_joint">
             <command_interface name="position" />
             <command_interface name="velocity" />
@@ -55,5 +95,5 @@
             <state_interface name="effort" />
         </joint>
-        <joint name="FL_calf_joint">
+        <joint name="HL_abd_joint">
             <command_interface name="position" />
             <command_interface name="velocity" />
@@ -65,5 +105,5 @@
             <state_interface name="effort" />
         </joint>
-        <joint name="RR_hip_joint">
+        <joint name="HL_hip_joint">
             <command_interface name="position" />
             <command_interface name="velocity" />
@@ -75,45 +115,5 @@
             <state_interface name="effort" />
         </joint>
-        <joint name="RR_thigh_joint">
-            <command_interface name="position" />
-            <command_interface name="velocity" />
-            <command_interface name="effort" />
-            <command_interface name="kp" />
-            <command_interface name="kd" />
-            <state_interface name="position" />
-            <state_interface name="velocity" />
-            <state_interface name="effort" />
-        </joint>
-        <joint name="RR_calf_joint">
-            <command_interface name="position" />
-            <command_interface name="velocity" />
-            <command_interface name="effort" />
-            <command_interface name="kp" />
-            <command_interface name="kd" />
-            <state_interface name="position" />
-            <state_interface name="velocity" />
-            <state_interface name="effort" />
-        </joint>
-        <joint name="RL_hip_joint">
-            <command_interface name="position" />
-            <command_interface name="velocity" />
-            <command_interface name="effort" />
-            <command_interface name="kp" />
-            <command_interface name="kd" />
-            <state_interface name="position" />
-            <state_interface name="velocity" />
-            <state_interface name="effort" />
-        </joint>
-        <joint name="RL_thigh_joint">
-            <command_interface name="position" />
-            <command_interface name="velocity" />
-            <command_interface name="effort" />
-            <command_interface name="kp" />
-            <command_interface name="kd" />
-            <state_interface name="position" />
-            <state_interface name="velocity" />
-            <state_interface name="effort" />
-        </joint>
-        <joint name="RL_calf_joint">
+        <joint name="HL_knee_joint">
             <command_interface name="position" />
             <command_interface name="velocity" />
