Commit message: 更新URDF命名规则

File: robot_description/galileo_mini_description/urdf/robot.urdf (robot description, URDF)
Before this commit: robot galileo_mini_description, 18 links, 17 joints
Links:
- removed link FL_calf
- removed link FL_foot
- removed link FL_hip
- removed link FL_thigh
- removed link FR_calf
- removed link FR_foot
- removed link FR_hip
- removed link FR_thigh
- removed link RL_calf
- removed link RL_foot
- removed link RL_hip
- removed link RL_thigh
- removed link RR_calf
- removed link RR_foot
- removed link RR_hip
- removed link RR_thigh
- removed link trunk
- added link FL_abd_link, mass 2.86; collision cylinder length=0.1065 radius=0.06; visual mesh filename=package://galileo_mini_description/meshes/FL_abd_link.STL
- added link FL_foot_link, mass 0.00020487; collision sphere radius=0.030; visual sphere radius=0.030
- added link FL_hip_link, mass 2.6; collision box size=0.06 0.035 0.26; visual mesh filename=package://galileo_mini_description/meshes/FL_hip_link.STL
- added link FL_knee_link, mass 0.314; collision box size=0.05 0.03 0.23; visual mesh filename=package://galileo_mini_description/meshes/FL_knee_link.STL
- added link FR_abd_link, mass 2.86; collision cylinder length=0.1065 radius=0.06; visual mesh filename=package://galileo_mini_description/meshes/FR_abd_link.STL
- added link FR_foot_link, mass 0.00020487; collision sphere radius=0.03; visual sphere radius=0.03
- added link FR_hip_link, mass 2.6; collision box size=0.06 0.035 0.26; visual mesh filename=package://galileo_mini_description/meshes/FR_hip_link.STL
- added link FR_knee_link, mass 0.314; collision box size=0.05 0.03 0.23; visual mesh filename=package://galileo_mini_description/meshes/FR_knee_link.STL
- added link HL_abd_link, mass 2.86; collision cylinder length=0.1065 radius=0.06; visual mesh filename=package://galileo_mini_description/meshes/HL_abd_link.STL
- added link HL_foot_link, mass 0.000204873572147578; collision sphere radius=0.03; visual sphere radius=0.03
- added link HL_hip_link, mass 2.6; collision box size=0.06 0.035 0.26; visual mesh filename=package://galileo_mini_description/meshes/HL_hip_link.STL
- added link HL_knee_link, mass 0.314; collision box size=0.05 0.03 0.23; visual mesh filename=package://galileo_mini_description/meshes/HL_knee_link.STL
- added link HR_abd_link, mass 2.86; collision cylinder length=0.1065 radius=0.06; visual mesh filename=package://galileo_mini_description/meshes/HR_abd_link.STL
- added link HR_foot_link, mass 0.000204873572147578; collision sphere radius=0.03; visual sphere radius=0.03
- added link HR_hip_link, mass 2.6; collision box size=0.06 0.035 0.26; visual mesh filename=package://galileo_mini_description/meshes/HR_hip_link.STL
- added link HR_knee_link, mass 0.314; collision box size=0.05 0.03 0.23; visual mesh filename=package://galileo_mini_description/meshes/HR_knee_link.STL
- added link base_link, mass 20.8; collision box size=0.45 0.25 0.1; visual mesh filename=package://galileo_mini_description/meshes/base_link.STL
Joints:
- removed joint FL_calf_joint
- removed joint FL_thigh_joint
- removed joint FR_calf_joint
- removed joint FR_thigh_joint
- removed joint RL_calf_joint
- removed joint RL_foot_joint
- removed joint RL_hip_joint
- removed joint RL_thigh_joint
- removed joint RR_calf_joint
- removed joint RR_hip_joint
- removed joint RR_thigh_joint
- added joint FL_abd_joint: type revolute, parent base_link, child FL_abd_link, origin xyz=0.2015 0.08 0 rpy=0 0 0, axis 1 0 0, limit lower=-0.80285 upper=0.80285 effort=100 velocity=21
- added joint FL_knee_joint: type revolute, parent FL_hip_link, child FL_knee_link, origin xyz=0 0 -0.26 rpy=0 0 0, axis 0 1 0, limit lower=0.9163 upper=2.6965 effort=150 velocity=21
- added joint FR_abd_joint: type revolute, parent base_link, child FR_abd_link, origin xyz=0.2015 -0.08 0 rpy=0 0 0, axis 1 0 0, limit lower=-0.80285 upper=0.80285 effort=100 velocity=21
- added joint FR_knee_joint: type revolute, parent FR_hip_link, child FR_knee_link, origin xyz=0 0 -0.26 rpy=0 0 0, axis 0 1 0, limit lower=0.9163 upper=2.6965 effort=150 velocity=21
- added joint HL_abd_joint: type revolute, parent base_link, child HL_abd_link, origin xyz=-0.2015 0.08 0 rpy=0 0 0, axis 1 0 0, limit lower=-0.80285 upper=0.80285 effort=100 velocity=21
- added joint HL_foot_link: type fixed, parent HL_knee_link, child HL_foot_link, origin xyz=0.0329385085367515 0 -0.261492891464613 rpy=0 0 0, axis 0 0 0
- added joint HL_hip_joint: type revolute, parent HL_abd_link, child HL_hip_link, origin xyz=-0.1 0.1065 0 rpy=0 0 0, axis 0 1 0, limit lower=-1.0472 upper=4.1888 effort=100 velocity=21
- added joint HL_knee_joint: type revolute, parent HL_hip_link, child HL_knee_link, origin xyz=6.3209E-05 0 -0.26 rpy=0 0 0, axis 0 1 0, limit lower=0.9163 upper=2.6965 effort=150 velocity=21
- added joint HR_abd_joint: type revolute, parent base_link, child HR_abd_link, origin xyz=-0.2015 -0.08 0 rpy=0 0 0, axis 1 0 0, limit lower=-0.80285 upper=0.80285 effort=100 velocity=21
- added joint HR_hip_joint: type revolute, parent HR_abd_link, child HR_hip_link, origin xyz=-0.1 -0.10685 0 rpy=0 0 0, axis 0 1 0, limit lower=-1.0472 upper=4.1888 effort=100 velocity=21
- added joint HR_knee_joint: type revolute, parent HR_hip_link, child HR_knee_link, origin xyz=0 0 -0.26 rpy=0 0 0, axis 0 1 0, limit lower=0.9163 upper=2.6965 effort=150 velocity=21
- joint FL_foot_joint: child FL_foot -> FL_foot_link; parent FL_calf -> FL_knee_link
- joint FL_hip_joint: axis 1 0 0 -> 0 1 0; child FL_hip -> FL_hip_link; limit lower=-0.80285 upper=0.80285 effort=100 velocity=21 -> lower=-1.0472 upper=4.1888 effort=100 velocity=21; origin xyz=0.2015 0.08 0 rpy=0 0 0 -> xyz=0.1 0.1065 0 rpy=0 0 0; parent trunk -> FL_abd_link
- joint FR_foot_joint: child FR_foot -> FR_foot_link; parent FR_calf -> FR_knee_link
- joint FR_hip_joint: axis 1 0 0 -> 0 1 0; child FR_hip -> FR_hip_link; limit lower=-0.80285 upper=0.80285 effort=100 velocity=21 -> lower=-1.0472 upper=4.1888 effort=100 velocity=21; origin xyz=0.2015 -0.08 0 rpy=0 0 0 -> xyz=0.1 -0.10685 0 rpy=0 0 0; parent trunk -> FR_abd_link
- joint RR_foot_joint: child RR_foot -> HR_foot_link; parent RR_calf -> HR_knee_link
- joint floating_base_joint: child trunk -> base_link

File: robot_description/galileo_mini_description/xacro/robot.xacro (robot description, xacro)
@@ -7,7 +7,7 @@
     <origin xyz="0 0 0" rpy="0 0 0" />
     <parent link="base" />
-    <child link="trunk" />
-  </joint>
-  <link name="trunk">
+    <child link="base_link" />
+  </joint>
+  <link name="base_link">
     <inertial>
       <origin
@@ -30,5 +30,5 @@
       <geometry>
         <mesh
-          filename="package://galileo_mini_description/meshes/trunk.STL" />
+          filename="package://galileo_mini_description/meshes/base_link.STL" />
       </geometry>
       <material
@@ -46,5 +46,5 @@
     </collision>
   </link>
-  <link name="FL_hip">
+  <link name="FL_abd_link">
     <inertial>
       <origin
@@ -67,5 +67,5 @@
       <geometry>
         <mesh
-          filename="package://galileo_mini_description/meshes/FL_hip.STL" />
+          filename="package://galileo_mini_description/meshes/FL_abd_link.STL" />
       </geometry>
       <material
@@ -84,12 +84,12 @@
     </collision>
   </link>
-  <joint name="FL_hip_joint" type="revolute">
+  <joint name="FL_abd_joint" type="revolute">
     <origin
       xyz="0.2015 0.08 0"
       rpy="0 0 0" />
     <parent
-      link="trunk" />
-    <child
-      link="FL_hip" />
+      link="base_link" />
+    <child
+      link="FL_abd_link" />
     <axis
       xyz="1 0 0" />
@@ -100,5 +100,5 @@
       velocity="21" />
   </joint>
-  <link name="FL_thigh">
+  <link name="FL_hip_link">
     <inertial>
       <origin
@@ -121,5 +121,5 @@
       <geometry>
         <mesh
-          filename="package://galileo_mini_description/meshes/FL_thigh.STL" />
+          filename="package://galileo_mini_description/meshes/FL_hip_link.STL" />
       </geometry>
       <material
@@ -138,12 +138,12 @@
     </collision>
   </link>
-  <joint name="FL_thigh_joint" type="revolute">
+  <joint name="FL_hip_joint" type="revolute">
     <origin
       xyz="0.1 0.1065 0"
       rpy="0 0 0" />
     <parent
-      link="FL_hip" />
-    <child
-      link="FL_thigh" />
+      link="FL_abd_link" />
+    <child
+      link="FL_hip_link" />
     <axis
       xyz="0 1 0" />
@@ -154,5 +154,5 @@
       velocity="21" />
   </joint>
-  <link name="FL_calf">
+  <link name="FL_knee_link">
     <inertial>
       <origin
@@ -175,5 +175,5 @@
       <geometry>
         <mesh
-          filename="package://galileo_mini_description/meshes/FL_calf.STL" />
+          filename="package://galileo_mini_description/meshes/FL_knee_link.STL" />
       </geometry>
       <material
@@ -192,12 +192,12 @@
     </collision>
   </link>
-  <joint name="FL_calf_joint" type="revolute">
+  <joint name="FL_knee_joint" type="revolute">
     <origin
       xyz="0 0 -0.26"
       rpy="0 0 0" />
     <parent
-      link="FL_thigh" />
-    <child
-      link="FL_calf" />
+      link="FL_hip_link" />
+    <child
+      link="FL_knee_link" />
     <axis
       xyz="0 1 0" />
@@ -208,5 +208,5 @@
       velocity="21" />
   </joint>
-  <link name="FL_foot">
+  <link name="FL_foot_link">
     <inertial>
       <origin
@@ -250,18 +250,18 @@
       rpy="0 0 0" />
     <parent
-      link="FL_calf" />
-    <child
-      link="FL_foot" />
+      link="FL_knee_link" />
+    <child
+      link="FL_foot_link" />
     <axis
       xyz="0 0 0" />
   </joint>
-  <joint name="FR_hip_joint" type="revolute">
+  <joint name="FR_abd_joint" type="revolute">
     <origin
       xyz="0.2015 -0.08 0"
       rpy="0 0 0" />
     <parent
-      link="trunk" />
-    <child
-      link="FR_hip" />
+      link="base_link" />
+    <child
+      link="FR_abd_link" />
     <axis
       xyz="1 0 0" />
@@ -272,5 +272,5 @@
       velocity="21" />
   </joint>
-  <link name="FR_hip">
+  <link name="FR_abd_link">
     <inertial>
       <origin
@@ -293,5 +293,5 @@
       <geometry>
         <mesh
-          filename="package://galileo_mini_description/meshes/FR_hip.STL" />
+          filename="package://galileo_mini_description/meshes/FR_abd_link.STL" />
       </geometry>
       <material
@@ -310,12 +310,12 @@
     </collision>
   </link>
-  <joint name="FR_thigh_joint" type="revolute">
+  <joint name="FR_hip_joint" type="revolute">
     <origin
       xyz="0.1 -0.10685 0"
       rpy="0 0 0" />
     <parent
-      link="FR_hip" />
-    <child
-      link="FR_thigh" />
+      link="FR_abd_link" />
+    <child
+      link="FR_hip_link" />
     <axis
       xyz="0 1 0" />
@@ -326,5 +326,5 @@
       velocity="21" />
   </joint>
-  <link name="FR_thigh">
+  <link name="FR_hip_link">
     <inertial>
       <origin
@@ -347,5 +347,5 @@
       <geometry>
         <mesh
-          filename="package://galileo_mini_description/meshes/FR_thigh.STL" />
+          filename="package://galileo_mini_description/meshes/FR_hip_link.STL" />
       </geometry>
       <material
@@ -364,12 +364,12 @@
     </collision>
   </link>
-  <joint name="FR_calf_joint" type="revolute">
+  <joint name="FR_knee_joint" type="revolute">
     <origin
       xyz="0 0 -0.26"
       rpy="0 0 0" />
     <parent
-      link="FR_thigh" />
-    <child
-      link="FR_calf" />
+      link="FR_hip_link" />
+    <child
+      link="FR_knee_link" />
     <axis
       xyz="0 1 0" />
@@ -380,5 +380,5 @@
       velocity="21" />
   </joint>
-  <link name="FR_calf">
+  <link name="FR_knee_link">
     <inertial>
       <origin
@@ -401,5 +401,5 @@
       <geometry>
         <mesh
-          filename="package://galileo_mini_description/meshes/FR_calf.STL" />
+          filename="package://galileo_mini_description/meshes/FR_knee_link.STL" />
       </geometry>
       <material
@@ -423,11 +423,11 @@
       rpy="0 0 0" />
     <parent
-      link="FR_calf" />
-    <child
-      link="FR_foot" />
+      link="FR_knee_link" />
+    <child
+      link="FR_foot_link" />
     <axis
       xyz="0 0 0" />
   </joint>
-  <link name="FR_foot">
+  <link name="FR_foot_link">
     <inertial>
       <origin
@@ -466,12 +466,12 @@
     </collision>
   </link>
-  <joint name="RR_hip_joint" type="revolute">
+  <joint name="HR_abd_joint" type="revolute">
     <origin
       xyz="-0.2015 -0.08 0"
       rpy="0 0 0" />
     <parent
-      link="trunk" />
-    <child
-      link="RR_hip" />
+      link="base_link" />
+    <child
+      link="HR_abd_link" />
     <axis
       xyz="1 0 0" />
@@ -482,5 +482,5 @@
       velocity="21" />
   </joint>
-  <link name="RR_hip">
+  <link name="HR_abd_link">
     <inertial>
       <origin
@@ -503,5 +503,5 @@
       <geometry>
         <mesh
-          filename="package://galileo_mini_description/meshes/RR_hip.STL" />
+          filename="package://galileo_mini_description/meshes/HR_abd_link.STL" />
       </geometry>
       <material
@@ -520,12 +520,12 @@
     </collision>
   </link>
-  <joint name="RR_thigh_joint" type="revolute">
+  <joint name="HR_hip_joint" type="revolute">
     <origin
       xyz="-0.1 -0.10685 0"
       rpy="0 0 0" />
     <parent
-      link="RR_hip" />
-    <child
-      link="RR_thigh" />
+      link="HR_abd_link" />
+    <child
+      link="HR_hip_link" />
     <axis
       xyz="0 1 0" />
@@ -536,5 +536,5 @@
       velocity="21" />
   </joint>
-  <link name="RR_thigh">
+  <link name="HR_hip_link">
     <inertial>
       <origin
@@ -557,5 +557,5 @@
       <geometry>
         <mesh
-          filename="package://galileo_mini_description/meshes/RR_thigh.STL" />
+          filename="package://galileo_mini_description/meshes/HR_hip_link.STL" />
       </geometry>
       <material
@@ -574,12 +574,12 @@
     </collision>
   </link>
-  <joint name="RR_calf_joint" type="revolute">
+  <joint name="HR_knee_joint" type="revolute">
     <origin
       xyz="0 0 -0.26"
       rpy="0 0 0" />
     <parent
-      link="RR_thigh" />
-    <child
-      link="RR_calf" />
+      link="HR_hip_link" />
+    <child
+      link="HR_knee_link" />
     <axis
       xyz="0 1 0" />
@@ -590,5 +590,5 @@
       velocity="21" />
   </joint>
-  <link name="RR_calf">
+  <link name="HR_knee_link">
     <inertial>
       <origin
@@ -611,5 +611,5 @@
       <geometry>
         <mesh
-          filename="package://galileo_mini_description/meshes/RR_calf.STL" />
+          filename="package://galileo_mini_description/meshes/HR_knee_link.STL" />
       </geometry>
       <material
@@ -633,11 +633,11 @@
       rpy="0 0 0" />
     <parent
-      link="RR_calf" />
-    <child
-      link="RR_foot" />
+      link="HR_knee_link" />
+    <child
+      link="HR_foot_link" />
     <axis
       xyz="0 0 0" />
   </joint>
-  <link name="RR_foot">
+  <link name="HR_foot_link">
     <inertial>
       <origin
@@ -676,12 +676,12 @@
     </collision>
   </link>
-  <joint name="RL_hip_joint" type="revolute">
+  <joint name="HL_abd_joint" type="revolute">
     <origin
       xyz="-0.2015 0.08 0"
       rpy="0 0 0" />
     <parent
-      link="trunk" />
-    <child
-      link="RL_hip" />
+      link="base_link" />
+    <child
+      link="HL_abd_link" />
     <axis
       xyz="1 0 0" />
@@ -692,5 +692,5 @@
       velocity="21" />
   </joint>
-  <link name="RL_hip">
+  <link name="HL_abd_link">
     <inertial>
       <origin
@@ -713,5 +713,5 @@
       <geometry>
         <mesh
-          filename="package://galileo_mini_description/meshes/RL_hip.STL" />
+          filename="package://galileo_mini_description/meshes/HL_abd_link.STL" />
       </geometry>
       <material
@@ -730,12 +730,12 @@
     </collision>
   </link>
-  <joint name="RL_thigh_joint" type="revolute">
+  <joint name="HL_hip_joint" type="revolute">
     <origin
       xyz="-0.1 0.1065 0"
       rpy="0 0 0" />
     <parent
-      link="RL_hip" />
-    <child
-      link="RL_thigh" />
+      link="HL_abd_link" />
+    <child
+      link="HL_hip_link" />
     <axis
       xyz="0 1 0" />
@@ -746,5 +746,5 @@
       velocity="21" />
   </joint>
-  <link name="RL_thigh">
+  <link name="HL_hip_link">
     <inertial>
       <origin
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
File: robot_description/galileo_mini_description/xacro/ros2_control.xacro (robot description, xacro)
@@ -5,4 +5,14 @@
             <plugin>hardware_mujoco/HardwareMujoco</plugin>
         </hardware>
+        <joint name="FR_abd_joint">
+            <command_interface name="position" />
+            <command_interface name="velocity" />
+            <command_interface name="effort" />
+            <command_interface name="kp" />
+            <command_interface name="kd" />
+            <state_interface name="position" />
+            <state_interface name="velocity" />
+            <state_interface name="effort" />
+        </joint>
         <joint name="FR_hip_joint">
             <command_interface name="position" />
@@ -15,5 +25,5 @@
             <state_interface name="effort" />
         </joint>
-        <joint name="FR_thigh_joint">
+        <joint name="FR_knee_joint">
             <command_interface name="position" />
             <command_interface name="velocity" />
@@ -25,5 +35,5 @@
             <state_interface name="effort" />
         </joint>
-        <joint name="FR_calf_joint">
+        <joint name="FL_abd_joint">
             <command_interface name="position" />
             <command_interface name="velocity" />
@@ -45,5 +55,5 @@
             <state_interface name="effort" />
         </joint>
-        <joint name="FL_thigh_joint">
+        <joint name="FL_knee_joint">
             <command_interface name="position" />
             <command_interface name="velocity" />
@@ -55,5 +65,5 @@
             <state_interface name="effort" />
         </joint>
-        <joint name="FL_calf_joint">
+        <joint name="HR_abd_joint">
             <command_interface name="position" />
             <command_interface name="velocity" />
@@ -65,5 +75,5 @@
             <state_interface name="effort" />
         </joint>
-        <joint name="RR_hip_joint">
+        <joint name="HR_hip_joint">
             <command_interface name="position" />
             <command_interface name="velocity" />
@@ -75,5 +85,5 @@
             <state_interface name="effort" />
         </joint>
-        <joint name="RR_thigh_joint">
+        <joint name="HR_knee_joint">
             <command_interface name="position" />
             <command_interface name="velocity" />
@@ -85,5 +95,5 @@
             <state_interface name="effort" />
         </joint>
-        <joint name="RR_calf_joint">
+        <joint name="HL_abd_joint">
             <command_interface name="position" />
             <command_interface name="velocity" />
@@ -95,5 +105,5 @@
             <state_interface name="effort" />
         </joint>
-        <joint name="RL_hip_joint">
+        <joint name="HL_hip_joint">
             <command_interface name="position" />
             <command_interface name="velocity" />
@@ -105,15 +115,5 @@
             <state_interface name="effort" />
         </joint>
-        <joint name="RL_thigh_joint">
-            <command_interface name="position" />
-            <command_interface name="velocity" />
-            <command_interface name="effort" />
-            <command_interface name="kp" />
-            <command_interface name="kd" />
-            <state_interface name="position" />
-            <state_interface name="velocity" />
-            <state_interface name="effort" />
-        </joint>
-        <joint name="RL_calf_joint">
+        <joint name="HL_knee_joint">
             <command_interface name="position" />
             <command_interface name="velocity" />
@@ -138,8 +138,8 @@
         </sensor>
         <!-- <sensor name="foot_contact_sensor">
-            <state_interface name="FR_foot" />
-            <state_interface name="FL_foot" />
-            <state_interface name="RR_foot" />
-            <state_interface name="RL_foot" />
+            <state_interface name="FR_foot_link" />
+            <state_interface name="FL_foot_link" />
+            <state_interface name="HR_foot_link" />
+            <state_interface name="HL_foot_link" />
         </sensor> -->
     </ros2_control>

Commit message: 增加逆运动学关节空间跟踪

File: robot_description/galileo_mini_description/urdf/robot.urdf (robot description, URDF)
Before this commit: robot galileo_mini_description, 18 links, 17 joints
Links:
- removed link world
Joints:
- removed joint floating_base_joint
- joint FL_knee_joint: limit lower=0.9163 upper=2.6965 effort=150 velocity=21 -> lower=-2.6965 upper=-0.9163 effort=150 velocity=21
- joint FR_knee_joint: limit lower=0.9163 upper=2.6965 effort=150 velocity=21 -> lower=-2.6965 upper=-0.9163 effort=150 velocity=21
- joint HL_knee_joint: limit lower=0.9163 upper=2.6965 effort=150 velocity=21 -> lower=-2.6965 upper=-0.9163 effort=150 velocity=21
- joint HR_knee_joint: limit lower=0.9163 upper=2.6965 effort=150 velocity=21 -> lower=-2.6965 upper=-0.9163 effort=150 velocity=21

Commit message: 修正urdf中的限位

File: robot_description/galileo_mini_description/urdf/robot.urdf (robot description, URDF)
Before this commit: robot galileo_mini_description, 17 links, 16 joints
Joints:
- joint FL_hip_joint: limit lower=-1.0472 upper=4.1888 effort=100 velocity=21 -> lower=-4.1888 upper=1.0472 effort=100 velocity=21
- joint FR_hip_joint: limit lower=-1.0472 upper=4.1888 effort=100 velocity=21 -> lower=-4.1888 upper=1.0472 effort=100 velocity=21
- joint HL_hip_joint: limit lower=-1.0472 upper=4.1888 effort=100 velocity=21 -> lower=-4.1888 upper=1.0472 effort=100 velocity=21
- joint HR_hip_joint: limit lower=-1.0472 upper=4.1888 effort=100 velocity=21 -> lower=-4.1888 upper=1.0472 effort=100 velocity=21

Commit message: 修正URDF的命名BUG

File: robot_description/galileo_mini_description/urdf/robot.urdf (robot description, URDF)
Before this commit: robot galileo_mini_description, 17 links, 16 joints
Joints:
- removed joint RR_foot_joint
- added joint HR_foot_joint: type fixed, parent HR_knee_link, child HR_foot_link, origin xyz=0.032939 0 -0.26149 rpy=0 0 0, axis 0 0 0
